File: EE/500308-A_PCBA-TUB/500308-A_PCBA-TUB.kicad_pcb (KiCad board)
At the start: 4 copper layers, 60 x 60 mm, 91 parts, among them J1 Conn_01x05_Pin, Q1 DMN2075U, Q10 DMN2075U, Q11 DMN2075U, Q12 DMN2075U, Q13 DMN2075U, Q14 DMN2075U, Q2 DMN2075U, Q3 DMN2075U, Q4 DMN2075U, Q5 DMN2075U, Q6 DMN2075U, Q7 DMN2075U, Q8 DMN2075U, Q9 DMN2075U, U1 PCA9548ARGE, U10 TMP117xxYBG, U11 TMP117xxYBG, U12 TMP117xxYBG, U13 TMP117xxYBG, U14 TMP117xxYBG, U15 TMP117xxYBG, U16 TMP117xxYBG, U2 PCA9685BS, U3 TMP117xxYBG, U4 TMP117xxYBG, U5 TMP117xxYBG, U6 TMP117xxYBG, U7 TMP117xxYBG, U8 TMP117xxYBG, U9 TMP117xxYBG

Commit message: Only tmp sensors on well side
Parts:
- removed the C14 at (80.5, 87.0)
- removed J1: Conn_01x05_Pin, Connector_PinHeader_2.54mm:PinHeader_1x05_P2.54mm_Vertical
- added C1: .1uF, Capacitor_SMD:C_0402_1005Metric_Pad0.74x0.62mm_HandSolder, B.Cu at (76.8, 96.8)
- added J2: 53398-0571, Library:53398-0571, B.Cu at (90.4, 129.5)
- C10, C11, C12, C13, C15, C16, C2, C3, C4, C5, C6, C7, C8, C9, R43, R44, U1, U2: moved to B.Cu
- C14: renamed from C1; moved to B.Cu
- moved R43 13.4 mm to (101.1, 130.8), turned to -90 degrees
- moved C14 10.4 mm to (80.5, 87.0), turned to -25.7141 degrees
- moved R44 9.16 mm to (102.3, 132.2), turned to 90 degrees
- moved C15 8.37 mm to (77.4, 122.0), turned to 90 degrees
- moved C16 2.82 mm to (120.8, 122.6), turned to 0 degrees
- turned C10 to -128.571 degrees
- turned C11 to -102.857 degrees
- turned C12 to -77.1427 degrees
- turned C13 to -51.4284 degrees
- turned C2 to 25.7143 degrees
- turned C3 to 51.4286 degrees
- turned C4 to 77.1429 degrees
- turned C5 to 102.857 degrees
- turned C6 to 128.571 degrees
- turned C7 to 154.286 degrees
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Connections:
- R43 pad 1: /SCL -> /SDA
- R44 pad 1: /SDA -> /SCL
Routing:
- net /SCL: track 48.4 -> 69.0 mm
- net /SDA: track 48.1 -> 63.9 mm, vias 1 -> 2
- net /tmp117_array/SDA0: track 27.7 -> 15.0 mm
- net /Heaters/PWM_6: track 30.8 -> 39.2 mm, vias 2 -> 3
- net /tmp117_array/SCL0: track 35.4 -> 27.6 mm, vias 0 -> 1
- net /Heaters/PWM_5: track 24.5 -> 32.0 mm, vias 2 -> 3
- net /Heaters/PWM_7: track 38.1 -> 45.6 mm, vias 2 -> 3
- net /Heaters/PWM_10: track 55.7 -> 62.2 mm, vias 2 -> 3
- net /tmp117_array/SCL3: track 47.4 -> 53.9 mm, vias 2 -> 3
- net /Heaters/PWM_8: track 43.2 -> 49.6 mm, vias 2 -> 3
- net /Heaters/PWM_9: track 49.5 -> 55.8 mm, vias 2 -> 3
- net /tmp117_array/SDA3: track 40.8 -> 47.1 mm, vias 2 -> 3
- net +3V3: track 63.1 -> 58.6 mm, vias 23 -> 24
- net /tmp117_array/SCL2: track 81.7 -> 86.1 mm, vias 2 -> 3
- net /Heaters/PWM_4: track 25.3 -> 21.3 mm
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