File: EE/500308-A_PCBA-TUB/500308-A_PCBA-TUB.kicad_sch (KiCad schematic)
At the start: 7 parts, among them J1 Conn_01x05_Pin, U1 PCA9548ARGE, U2 PCA9685BS

Commit message: Only tmp sensors on well side
Parts:
- removed J1: Conn_01x05_Pin, Connector_PinHeader_2.54mm:PinHeader_1x05_P2.54mm_Vertical, symbol Connector:Conn_01x05_Pin
- added J2: 53398-0571, Library:53398-0571, symbol 53398-0571:53398-0571
Connections:
- net +12V: now also J2.1
- net +3V3: now also J2.2
- net GND: now also J2.3
- net SCL: now also R44.1, J2.4; no longer R43.1
- net SDA: now also R43.1, J2.5; no longer R44.1
Changed lines of the file:
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@@
-	)
-	(junction
-		(at 82.55 163.83)
-		(diameter 0)
-		(color 0 0 0 0)
 	)
 	(junction
@@
 	)
 	(junction
-		(at 90.17 166.37)
-		(diameter 0)
-		(color 0 0 0 0)
-	)
-	(junction
 		(at 82.55 152.4)
 		(diameter 0)
@@
 	(wire
 		(pts
+			(xy 34.29 165.1) (xy 34.29 158.75)
+		)
+		(stroke
+			(width 0)
+			(type default)
+		)
+	)
+	(wire
+		(pts
 			(xy 52.07 97.79) (xy 52.07 113.03)
 		)
@@
 	(wire
 		(pts
+			(xy 29.21 166.37) (xy 90.17 166.37)
+		)
+		(stroke
+			(width 0)
+			(type default)
+		)
+	)
+	(wire
+		(pts
 			(xy 177.8 40.64) (xy 177.8 45.72)
 		)
@@
 	(wire
 		(pts
-			(xy 82.55 163.83) (xy 97.79 163.83)
-		)
-		(stroke
-			(width 0)
-			(type default)
-		)
-	)
-	(wire
-		(pts
 			(xy 165.1 53.34) (xy 165.1 55.88)
 		)
@@
 	(wire
 		(pts
-			(xy 90.17 166.37) (xy 97.79 166.37)
+			(xy 29.21 166.37) (xy 29.21 156.21)
 		)
 		(stroke
@@
 	(wire
 		(pts
-			(xy 82.55 162.56) (xy 82.55 163.83)
+			(xy 82.55 162.56) (xy 82.55 165.1)
 		)
 		(stroke
@@
 	(wire
 		(pts
-			(xy 60.96 163.83) (xy 82.55 163.83)
-		)
-		(stroke
-			(width 0)
-			(type default)
-		)
-	)
-	(wire
-		(pts
 			(xy 195.58 69.85) (xy 207.01 69.85)
 		)
@@
 	(wire
 		(pts
-			(xy 60.96 166.37) (xy 90.17 166.37)
-		)
-		(stroke
-			(width 0)
-			(type default)
-		)
-	)
-	(wire
-		(pts
 			(xy 52.07 95.25) (xy 52.07 97.79)
 		)
@@
 	(wire
 		(pts
+			(xy 34.29 165.1) (xy 82.55 165.1)
+		)
+		(stroke
+			(width 0)
+			(type default)
+		)
+	)
+	(wire
+		(pts
 			(xy 52.07 113.03) (xy 64.77 113.03)
 		)
@@
 	(wire
 		(pts
+			(xy 34.29 158.75) (xy 40.64 158.75)
+		)
+		(stroke
+			(width 0)
+			(type default)
+		)
+	)
+	(wire
+		(pts
 			(xy 76.2 152.4) (xy 76.2 149.86)
 		)
@@
 		(pts
 			(xy 74.93 69.85) (xy 83.82 69.85)
+		)
+		(stroke
+			(width 0)
+			(type default)
+		)
+	)
+	(wire
+		(pts
+			(xy 29.21 156.21) (xy 40.64 156.21)
 		)
 		(stroke
@@
 	)
 	(label "SDA"
-		(at 48.26 69.85 0)
+		(at 34.29 158.75 0)
 		(effects
 			(font
@@
 	)
 	(label "SDA"
-		(at 97.79 166.37 0)
+		(at 48.26 69.85 0)
 		(effects
 			(font
@@
 	)
 	(label "SCL"
-		(at 97.79 163.83 0)
+		(at 34.29 156.21 0)
 		(effects
 			(font
@@
 	)
 	(symbol
-		(lib_id "Connector:Conn_01x05_Pin")
-		(at 55.88 161.29 0)
-		(unit 1)
-		(exclude_from_sim no)
-		(in_bom yes)
-		(on_board yes)
-		(dnp no)
-		(fields_autoplaced yes)
-		(property "Reference" "J1"
-			(at 56.515 151.13 0)
-			(effects
-				(font
-					(size 1.27 1.27)
-				)
-			)
-		)
-		(property "Value" "Conn_01x05_Pin"
-			(at 56.515 153.67 0)
-			(effects
-				(font
-					(size 1.27 1.27)
-				)
-			)
-		)
-		(property "Footprint" "Connector_PinHeader_2.54mm:PinHeader_1x05_P2.54mm_Vertical"
-			(at 55.88 161.29 0)
-			(effects
-				(font
-					(size 1.27 1.27)
-				)
-				(hide yes)
-			)
-		)
-		(property "Datasheet" "~"
-			(at 55.88 161.29 0)
-			(effects
-				(font
-					(size 1.27 1.27)
-				)
-				(hide yes)
-			)
-		)
-		(property "Description" "Generic connector, single row, 01x05, script generated"
-			(at 55.88 161.29 0)
-			(effects
-				(font
-					(size 1.27 1.27)
-				)
-				(hide yes)
-			)
-		)
-		(pin "4"
-		)
-		(pin "5"
-		)
-		(pin "2"
-		)
-		(pin "1"
-		)
-		(pin "3"
-		)
-		(instances
-			(project ""
-				(path "/3517744d-988e-4a4e-a0d2-68e8d779ca14"
-					(reference "J1")
-					(unit 1)
-				)
-			)
-		)
-	)
-	(symbol
 		(lib_id "Device:R")
 		(at 82.55 158.75 180)
@@
 					(unit 1)
 				)
+			)
+		)
+	)
+	(symbol
+		(lib_id "53398-0571:53398-0571")
+		(at 60.96 156.21 0)
+		(mirror y)
+		(unit 1)
+		(exclude_from_sim no)
+		(in_bom yes)
+		(on_board yes)
+		(dnp no)
+		(property "Reference" "J2"
+			(at 50.8 148.59 0)
+			(effects
+				(font
+					(size 1.27 1.27)
+				)
+			)
+		)
+		(property "Value" "53398-0571"
+			(at 50.8 151.13 0)
+			(effects
+				(font
+					(size 1.27 1.27)
+				)
+			)
+		)
+		(property "Footprint" "Library:53398-0571"
+			(at 44.45 251.13 0)
+			(effects
+				(font
+					(size 1.27 1.27)
+				)
+				(justify left top)
+				(hide yes)
+			)
+		)
+		(property "Datasheet" "http://www.molex.com/pdm_docs/sd/533980571_sd.pdf"
+			(at 44.45 351.13 0)
+			(effects
+				(font
+					(size 1.27 1.27)
+				)
+				(justify left top)
+				(hide yes)
+			)
+		)
+		(property "Description" "Molex PICOBLADE Series, Series Number 53398, 1.25mm Pitch 5 Way 1 Row Straight PCB Header, Solder Termination, 1A"
+			(at 60.96 156.21 0)
+			(effects
+				(font
+					(size 1.27 1.27)
+				)
+				(hide yes)
+			)
+		)
+		(property "Height" ""
+			(at 44.45 551.13 0)
+			(effects
+				(font
+					(size 1.27 1.27)
+				)
+				(justify left top)
+				(hide yes)
+			)
+		)
+		(property "Mouser Part Number" "538-53398-0571"
+			(at 44.45 651.13 0)
+			(effects
+				(font
+					(size 1.27 1.27)
+				)
+				(justify left top)
+				(hide yes)
+			)
+		)
+		(property "Mouser Price/Stock" "https://www.mouser.co.uk/ProductDetail/Molex/53398-0571?qs=yqtfsgZKt1Q%2F%2FuRD6tNN4w%3D%3D"
+			(at 44.45 751.13 0)
+			(effects
+				(font
+					(size 1.27 1.27)
+				)
+				(justify left top)
+				(hide yes)
+			)
+		)
+		(property "Manufacturer_Name" "Molex"
+			(at 44.45 851.13 0)
+			(effects
+				(font
+					(size 1.27 1.27)
+				)
+				(justify left top)
+				(hide yes)
+			)
+		)
+		(property "Manufacturer_Part_Number" "53398-0571"
+			(at 44.45 951.13 0)
+			(effects
+				(font
+					(size 1.27 1.27)
+				)
+				(justify left top)
+				(hide yes)
+			)
+		)
+		(pin "2"
+		)
+		(pin "1"
+		)
+		(pin "4"
+		)
+		(pin "5"
+		)
+		(pin "3"
+		)
+		(instances
+			(project ""
+				(path "/3517744d-988e-4a4e-a0d2-68e8d779ca14"
+					(reference "J2")
+					(unit 1)
+				)
